File: hardware/hardware.kicad_sch (KiCad schematic)
At the start: 43 parts, among them IC4 NE555, J1 Li-Po battery, J11 pin_2, J12 servo, J13 UART, J14 ultrasonic, J19 ESP, J2 Screw_Terminal_01x02, J3 5V_DC/DC, J4 Solar panel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

Commit message: nowa wersja
Parts:
- D9: value D_Zener -> 5.1 V
- J19: value ESP -> 5V_ESP
- J2: value Screw_Terminal_01x02 -> 5V_OUT
- R21: value R -> 220
Connections:
- net TRIG: now reaches C1.1, D7.1 (K), IC4.2 (~{TRIG}), IC4.6 (THRS), R2.1
Other:
- removed sheet esp+peryferia
- removed sheet zasilanie
- note added: "POWER SUPPLY BETWEEN PCB'S"
- note removed: "znalezc cewke i jej footprint a potem MOSFET"
- moved on the sheet: C2, D7, D9, IC4, J19, J2, J3, Q1, Q5, R1, R10, R11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
